Commit message: ...

File: description/hosbot_core.xacro (robot description, xacro)
@@ -159,3 +159,9 @@
         <material>Gazebo/Black</material>
     </gazebo>
+    <link   name =  "base_footprint"/>
+    <joint name = "base_joint"  type = "fixed">
+        <parent link="base_footprint"/>
+        <child link="base_link"/>
+        <origin xyz="0.0 0.0 0.0" rpy="0 0 0" />
+    </joint>
 </robot>
